File: Electronics/Lightbulb.brd (EAGLE design)
At the start: 61.5 x 47 mm, 19 parts, among them IC2 7805L

Commit message: updating a few resistor values for diodes to prevent draw of too much current from Arduino
Parts:
- R4: value 33Ω -> 47Ω
- R7: value 150Ω -> 100Ω
- R8, R9: value 100Ω -> 47Ω
Changed lines of the file:
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@@
 <attribute name="VALUE" x="57.151" y="11.358" size="1.27" layer="27" rot="R90"/>
 </element>
-<element name="R4" library="adafruit" package="R0805" value="33Ω" x="22.26" y="23.15">
+<element name="R4" library="adafruit" package="R0805" value="47Ω" x="22.26" y="23.15">
 <attribute name="NAME" x="21.498" y="24.166" size="1.27" layer="25"/>
 <attribute name="VALUE" x="21.498" y="20.864" size="1.27" layer="27"/>
@@
 <attribute name="VALUE" x="57.151" y="5.608" size="1.27" layer="27" rot="R90"/>
 </element>
-<element name="R7" library="adafruit" package="R0805" value="150Ω" x="23.53" y="10.1">
+<element name="R7" library="adafruit" package="R0805" value="100Ω" x="23.53" y="10.1">
 <attribute name="NAME" x="22.768" y="11.116" size="1.27" layer="25"/>
 <attribute name="VALUE" x="22.768" y="7.814" size="1.27" layer="27"/>
 </element>
-<element name="R8" library="adafruit" package="R0805" value="100Ω" x="23.53" y="15.48">
+<element name="R8" library="adafruit" package="R0805" value="47Ω" x="23.53" y="15.48">
 <attribute name="NAME" x="22.768" y="16.496" size="1.27" layer="25"/>
 <attribute name="VALUE" x="22.768" y="13.194" size="1.27" layer="27"/>
 </element>
-<element name="R9" library="adafruit" package="R0805" value="100Ω" x="23.53" y="4.72">
+<element name="R9" library="adafruit" package="R0805" value="47Ω" x="23.53" y="4.72">
 <attribute name="NAME" x="22.768" y="5.736" size="1.27" layer="25"/>
 <attribute name="VALUE" x="22.768" y="2.434" size="1.27" layer="27"/>
